File: KiCAD/ESP32WifiAisTempVolt2/ESP32WifiAisTempVolt2.kicad_pcb (KiCad board)
At the start: 2 copper layers, 80 x 54.9 mm, 18 parts, among them J1 Power, J2 D24V10F5, J3 AIS, J4 DS18B20, J5 CAN-Transceiver, Q1 BC547, Q2 BC547, SW1 SW_Push, U1 ESP32

Commit message: Version 1.1
Parts:
- J1, J3: footprint Connector_Wago:Wago_734-132_1x02_P3.50mm_Vertical -> TerminalBlock:TerminalBlock_bornier-2_P5.08mm
- J4: footprint Connector_Wago:Wago_734-133_1x03_P3.50mm_Vertical -> TerminalBlock:TerminalBlock_bornier-3_P5.08mm
- Q1, Q2: footprint Package_TO_SOT_THT:TO-92_Inline -> Package_TO_SOT_THT:TO-92_HandSolder
- moved J4 2.54 mm to (171.4, 94.0)
- moved J1 0.63 mm to (171.4, 76.8)
Connections:
- B1 pad 2: (no net) -> Net-(B1-Pad2)
- J2 pad 1: (no net) -> Net-(J2-Pad1)
- J2 pad 2: (no net) -> Net-(J2-Pad2)
- U1 pad 10: (no net) -> Net-(U1-Pad10)
- U1 pad 11: (no net) -> Net-(U1-Pad11)
- U1 pad 12: (no net) -> Net-(U1-Pad12)
- U1 pad 16: (no net) -> Net-(U1-Pad16)
- U1 pad 17: (no net) -> Net-(U1-Pad17)
- U1 pad 18: (no net) -> Net-(U1-Pad18)
- U1 pad 2: (no net) -> Net-(U1-Pad2)
- U1 pad 20: (no net) -> Net-(U1-Pad20)
- U1 pad 21: (no net) -> Net-(U1-Pad21)
- U1 pad 22: (no net) -> Net-(U1-Pad22)
- U1 pad 23: (no net) -> Net-(U1-Pad23)
- U1 pad 24: (no net) -> Net-(U1-Pad24)
- U1 pad 28: (no net) -> Net-(U1-Pad28)
- U1 pad 3: (no net) -> Net-(U1-Pad3)
- U1 pad 30: (no net) -> Net-(U1-Pad30)
- U1 pad 31: (no net) -> Net-(U1-Pad31)
- U1 pad 33: (no net) -> Net-(U1-Pad33)
- U1 pad 34: (no net) -> Net-(U1-Pad34)
- U1 pad 35: (no net) -> Net-(U1-Pad35)
- U1 pad 36: (no net) -> Net-(U1-Pad36)
- U1 pad 37: (no net) -> Net-(U1-Pad37)
- U1 pad 38: (no net) -> Net-(U1-Pad38)
- U1 pad 4: (no net) -> Net-(U1-Pad4)
- U1 pad 6: (no net) -> Net-(U1-Pad6)
- U1 pad 7: (no net) -> Net-(U1-Pad7)
- U1 pad 8: (no net) -> Net-(U1-Pad8)
- U1 pad 9: (no net) -> Net-(U1-Pad9)
Routing:
- net +3V3: track 105.0 -> 103.5 mm
- net GND: track 247.2 -> 248.6 mm
- net Net-(Q1-Pad2): track 7.93 -> 6.66 mm
Other:
- board text added: "+"
- board text added: "-"
- board text added: "NMEA2000 WiFi Gateway Rev 1.1"
- board text added: "S"
- board text removed: "NMEA2000 WiFi Gateway Rev 1.0"
